File: KiCAD/Keyboard.sch (KiCad schematic (older format))
At the start: 1 part

Commit message: Imported another KiCAD library Started with keyboard switches PCB design. Added another wishlist item.
Signed-off-by: itractus <karelclijsters@outlook.com>
Parts:
- removed U?: Teensy3.6, symbol Teensy3.6
- added 1!, A, CAPSlock, Escape, F1, K? (x6), LShift, Lctrl, Lsuper, Q, TAB, Tilde: KEYSW, symbol KEYSW
- added D? (x17): D_ALT, symbol D_ALT
Connections:
- wire segments 0 -> 89

Commit message: Completed keyboard layout. Added layout in jpeg for reference.
Signed-off-by: itractus <karelclijsters@outlook.com>
Parts:
- removed 1!, A, CAPSlock, Escape, F1, K? (x6), LShift, Lctrl, Lsuper, Q, TAB, Tilde: KEYSW, symbol KEYSW
- removed D? (x17): D_ALT, symbol D_ALT
- added D? (x101): D_ALT, symbol D_ALT
- added K? (x100), K??: KEYSW, symbol KEYSW
Connections:
- wire segments 89 -> 521
